Commit message: MOIRO Success Version

File: moiro_agv_description/urdf/moiro_agv.xacro (robot description, xacro)
@@ -11,5 +11,5 @@
     <origin xyz="0 0 0" rpy="0 0 0"/>
     <geometry>
-      <mesh filename="file://$(find moiro_agv_description)/meshes/base_link.stl" scale="0.001 0.001 0.001"/>
+      <mesh filename="package://moiro_agv_description/meshes/base_link.stl" scale="0.001 0.001 0.001"/>
     </geometry>
     <material name="silver"/>
